Commit message: Fix portable mesh resource URIs

File: urdf/base/base.urdf.xacro (robot description, xacro)
@@ -27,5 +27,5 @@
                 <origin xyz="0 0 0" rpy="0 0 0" />
                 <geometry>
-                    <mesh filename="file://$(find go2_description)/meshes/base/base.dae" scale="1 1 1"/>
+                    <mesh filename="package://go2_description/meshes/base/base.dae" scale="1 1 1"/>
                 </geometry>
                 <material
@@ -37,5 +37,5 @@
                 <origin xyz="0 0 0" rpy="0 0 0" />
                 <geometry>
-                    <mesh filename="file://$(find go2_description)/meshes/base/base.dae" scale="1 1 1"/>
+                    <mesh filename="package://go2_description/meshes/base/base.dae" scale="1 1 1"/>
                 </geometry>
             </collision>

File: urdf/leg/calf.urdf.xacro (robot description, xacro)
@@ -26,8 +26,8 @@
                 <geometry>
                     <xacro:unless value="${reflect}">
-                        <mesh filename="file://$(find go2_description)/meshes/leg/calf.dae" scale="1 1 1"/>
+                        <mesh filename="package://go2_description/meshes/leg/calf.dae" scale="1 1 1"/>
                     </xacro:unless>
                     <xacro:if value="${reflect}">
-                        <mesh filename="file://$(find go2_description)/meshes/leg/calf_mirror.dae" scale="1 1 1"/>
+                        <mesh filename="package://go2_description/meshes/leg/calf_mirror.dae" scale="1 1 1"/>
                     </xacro:if>
                 </geometry>
@@ -41,8 +41,8 @@
                 <geometry>
                     <xacro:unless value="${reflect}">
-                        <mesh filename="file://$(find go2_description)/meshes/leg/calf.dae" scale="1 1 1"/>
+                        <mesh filename="package://go2_description/meshes/leg/calf.dae" scale="1 1 1"/>
                     </xacro:unless>
                     <xacro:if value="${reflect}">
-                        <mesh filename="file://$(find go2_description)/meshes/leg/calf_mirror.dae" scale="1 1 1"/>
+                        <mesh filename="package://go2_description/meshes/leg/calf_mirror.dae" scale="1 1 1"/>
                     </xacro:if>
                 </geometry>

File: urdf/leg/foot.urdf.xacro (robot description, xacro)
@@ -19,5 +19,5 @@
                 <origin xyz="0 0 0" rpy="0 0 0" />
                 <geometry>
-                    <mesh filename="file://$(find go2_description)/meshes/leg/foot.dae" scale="1 1 1"/>
+                    <mesh filename="package://go2_description/meshes/leg/foot.dae" scale="1 1 1"/>
                 </geometry>
                 <material
@@ -29,5 +29,5 @@
                 <origin xyz="0 0 0" rpy="0 0 0" />
                 <geometry>
-                    <mesh filename="file://$(find go2_description)/meshes/leg/foot.dae" scale="1 1 1"/>
+                    <mesh filename="package://go2_description/meshes/leg/foot.dae" scale="1 1 1"/>
                 </geometry>
             </collision>

File: urdf/leg/hip.urdf.xacro (robot description, xacro)
@@ -31,5 +31,5 @@
                 <origin xyz="0 0 0" rpy="0 0 0" />
                 <geometry>
-                    <mesh filename="file://$(find go2_description)/meshes/leg/hip.dae" scale="1 1 1"/>
+                    <mesh filename="package://go2_description/meshes/leg/hip.dae" scale="1 1 1"/>
                 </geometry>
                 <material
@@ -41,5 +41,5 @@
                 <origin xyz="0 0 0" rpy="0 0 0" />
                 <geometry>
-                    <mesh filename="file://$(find go2_description)/meshes/leg/hip.dae" scale="1 1 1"/>
+                    <mesh filename="package://go2_description/meshes/leg/hip.dae" scale="1 1 1"/>
                 </geometry>
             </collision>

File: urdf/leg/thigh.urdf.xacro (robot description, xacro)
@@ -26,8 +26,8 @@
                 <geometry>
                     <xacro:unless value="${reflect}">
-                        <mesh filename="file://$(find go2_description)/meshes/leg/thigh.dae" scale="1 1 1"/>
+                        <mesh filename="package://go2_description/meshes/leg/thigh.dae" scale="1 1 1"/>
                     </xacro:unless>
                     <xacro:if value="${reflect}">
-                        <mesh filename="file://$(find go2_description)/meshes/leg/thigh_mirror.dae" scale="1 1 1"/>
+                        <mesh filename="package://go2_description/meshes/leg/thigh_mirror.dae" scale="1 1 1"/>
                     </xacro:if>
                 </geometry>
@@ -41,8 +41,8 @@
                 <geometry>
                     <xacro:unless value="${reflect}">
-                        <mesh filename="file://$(find go2_description)/meshes/leg/thigh.dae" scale="1 1 1"/>
+                        <mesh filename="package://go2_description/meshes/leg/thigh.dae" scale="1 1 1"/>
                     </xacro:unless>
                     <xacro:if value="${reflect}">
-                        <mesh filename="file://$(find go2_description)/meshes/leg/thigh_mirror.dae" scale="1 1 1"/>
+                        <mesh filename="package://go2_description/meshes/leg/thigh_mirror.dae" scale="1 1 1"/>
                     </xacro:if>
                 </geometry>

File: urdf/sensors/hesai.urdf.xacro (robot description, xacro)
@@ -11,5 +11,5 @@
             <visual>
                 <geometry>
-                    <mesh filename="file://$(find go2_description)/meshes/sensors/hesai_XT16.dae" scale="1 1 1"/>
+                    <mesh filename="package://go2_description/meshes/sensors/hesai_XT16.dae" scale="1 1 1"/>
                 </geometry>
                 <material name="">
@@ -19,5 +19,5 @@
             <collision>
                 <geometry>
-                    <mesh filename="file://$(find go2_description)/meshes/sensors/hesai_XT16.dae" scale="1 1 1"/>
+                    <mesh filename="package://go2_description/meshes/sensors/hesai_XT16.dae" scale="1 1 1"/>
                 </geometry>
             </collision>

Commit message: refactor: Remove fixed base_footprint from URDF

File: urdf/base/base.urdf.xacro (robot description, xacro)
@@ -3,17 +3,4 @@
     <!-- Define a macro for base_link -->
     <xacro:macro name="go2_base" params="prefix">
-        <link name="${prefix}base_footprint">
-            <visual>
-                <origin xyz="0 0 0" rpy="0 0 0" />
-                <geometry>
-                    <box size="0.001 0.001 0.001" />
-                </geometry>
-            </visual>
-        </link>
-		<joint name="${prefix}base_footprint_joint" type="fixed">
-            <origin xyz="0 0 0" rpy="0 0 0" /> <!-- A Z level is required -->
-            <parent link="${prefix}base_footprint"/>
-            <child link="${prefix}base_link" />
-		</joint>
         <link name="${prefix}base_link">
             <inertial>
