Commit message: fix: Remove white visual material overriding mesh colors
rviz_default_plugins 14.1.23 (ros2/rviz#1782) applies the URDF
<material> to every submesh when present, so the placeholder
rgba="1 1 1 1" turned the whole robot white. The DAE meshes carry
their own colors, so the tag is unnecessary.

Closes #14

Co-Authored-By: Claude Fable 5.1 <noreply@anthropic.com>

File: urdf/base/base.urdf.xacro (robot description, xacro)
@@ -16,8 +16,4 @@
                     <mesh filename="package://go2_description/meshes/base/base.dae" scale="1 1 1"/>
                 </geometry>
-                <material
-                    name="">
-                    <color rgba="1 1 1 1" />
-                </material>
             </visual>
             <collision>

File: urdf/leg/calf.urdf.xacro (robot description, xacro)
@@ -38,8 +38,4 @@
                     </xacro:if>
                 </geometry>
-                <material
-                    name="">
-                    <color rgba="1 1 1 1" />
-                </material>
             </visual>
             <collision>

File: urdf/leg/foot.urdf.xacro (robot description, xacro)
@@ -21,8 +21,4 @@
                     <mesh filename="package://go2_description/meshes/leg/foot.dae" scale="1 1 1"/>
                 </geometry>
-                <material
-                    name="">
-                    <color rgba="1 1 1 1" />
-                </material>
             </visual>
             <collision>

File: urdf/leg/hip.urdf.xacro (robot description, xacro)
@@ -46,8 +46,4 @@
                     <mesh filename="package://go2_description/meshes/leg/hip.dae" scale="1 1 1"/>
                 </geometry>
-                <material
-                    name="">
-                    <color rgba="1 1 1 1" />
-                </material>
             </visual>
             <collision>

File: urdf/leg/thigh.urdf.xacro (robot description, xacro)
@@ -47,8 +47,4 @@
                     </xacro:if>
                 </geometry>
-                <material
-                    name="">
-                    <color rgba="1 1 1 1" />
-                </material>
             </visual>
             <collision>

File: urdf/sensors/hesai.urdf.xacro (robot description, xacro)
@@ -13,7 +13,4 @@
                     <mesh filename="package://go2_description/meshes/sensors/hesai_XT16.dae" scale="1 1 1"/>
                 </geometry>
-                <material name="">
-                    <color rgba="1 1 1 1"/>
-                </material>
             </visual>
             <collision>
