Commit message: fix: Remove leg joint frame rotations

File: urdf/base/leg.urdf.xacro (robot description, xacro)
@@ -2,11 +2,7 @@
 <robot xmlns:xacro="http://ros.org/wiki/xacro">
 <xacro:include filename="$(find go2_description)/urdf/leg/hip.urdf.xacro"/>
-<xacro:property name="FL_" value="FL_" />
-<xacro:property name="FR_" value="FR_" />
-<xacro:property name="RL_" value="RL_" />
-<xacro:property name="RR_" value="RR_" />
-  <xacro:macro name="go2_leg" params="prefix parent reflect x y z roll pitch yaw">
-    <xacro:go2_hip prefix="${prefix}" parent="${parent}" reflect="${reflect}">
-      <origin xyz="${x} ${y} ${z}" rpy="${roll} ${pitch} ${yaw}"/>
+  <xacro:macro name="go2_leg" params="prefix parent front reflect x y z">
+    <xacro:go2_hip prefix="${prefix}" parent="${parent}" front="${front}" reflect="${reflect}">
+      <origin xyz="${x} ${y} ${z}" rpy="0 0 0"/>
     </xacro:go2_hip>
   </xacro:macro>

File: urdf/go2.urdf.xacro (robot description, xacro)
@@ -6,25 +6,20 @@
 <!-- Define a macro for the whole Go2 body (base + legs) -->
 <xacro:macro name="go2" params="prefix">
-    <!-- Global Properties  -->
-    <xacro:property name="PI" value="3.1415926535897931"/>
     <!-- Leg Allocations -->
-    <xacro:property name="leg_offset_x" value="0.194"/>
+    <xacro:property name="leg_offset_x" value="0.1934"/>
     <xacro:property name="leg_offset_y" value="0.0465"/>
     <xacro:property name="leg_offset_z" value="0.0"/>
     <!-- Robot base -->
     <xacro:go2_base prefix="${prefix}"/>
-    <!-- Legs -->
-    <xacro:go2_leg prefix="${prefix}FL_" parent="${prefix}base_link" reflect="false"
-            x="${leg_offset_x}"   y="${leg_offset_y}"   z="${leg_offset_z}"
-            roll="0"      pitch="0"   yaw="0"/>
-    <xacro:go2_leg prefix="${prefix}FR_" parent="${prefix}base_link" reflect="true"
-            x="${leg_offset_x}"   y="-${leg_offset_y}"  z="${leg_offset_z}"
-            roll="${PI}"  pitch="0"   yaw="0"/>
-    <xacro:go2_leg prefix="${prefix}RL_" parent="${prefix}base_link" reflect="false"
-            x="-${leg_offset_x}"  y="${leg_offset_y}"   z="${leg_offset_z}"
-            roll="${PI}"  pitch="0"   yaw="${PI}"/>
-    <xacro:go2_leg prefix="${prefix}RR_" parent="${prefix}base_link" reflect="true"
-            x="-${leg_offset_x}"  y="-${leg_offset_y}"  z="${leg_offset_z}"
-            roll="0"      pitch="0"   yaw="${PI}"/>
+    <!-- Legs: front/left flags select joint limits, inertia mirroring and meshes.
+         All joint origins are pure translations (no rotation), matching the real robot. -->
+    <xacro:go2_leg prefix="${prefix}FL_" parent="${prefix}base_link" front="true" reflect="false"
+            x="${leg_offset_x}"   y="${leg_offset_y}"   z="${leg_offset_z}"/>
+    <xacro:go2_leg prefix="${prefix}FR_" parent="${prefix}base_link" front="true" reflect="true"
+            x="${leg_offset_x}"   y="-${leg_offset_y}"  z="${leg_offset_z}"/>
+    <xacro:go2_leg prefix="${prefix}RL_" parent="${prefix}base_link" front="false" reflect="false"
+            x="-${leg_offset_x}"  y="${leg_offset_y}"   z="${leg_offset_z}"/>
+    <xacro:go2_leg prefix="${prefix}RR_" parent="${prefix}base_link" front="false" reflect="true"
+            x="-${leg_offset_x}"  y="-${leg_offset_y}"  z="${leg_offset_z}"/>
 </xacro:macro>
 </robot>

File: urdf/leg/hip.urdf.xacro (robot description, xacro)
@@ -3,13 +3,24 @@
 <xacro:include filename="$(find go2_description)/urdf/leg/thigh.urdf.xacro"/>
     <!-- Define a macro for hip -->
-    <xacro:macro name="go2_hip" params="prefix parent *origin reflect">
+    <xacro:macro name="go2_hip" params="prefix parent *origin front reflect">
         <xacro:property name="thigh_offset_x" value="0.0"/>
         <xacro:property name="thigh_offset_y" value="0.0955"/>
         <xacro:property name="thigh_offset_z" value="0.0"/>
-        <xacro:if value="${(prefix == RL_) or (prefix == RR_)}">
-            <xacro:property name="hip_angle" value="${PI}"/>
+        <!-- Mirror factors: y_sign flips left/right. The shared hip mesh is
+             reoriented per leg via the visual/collision origin only, so joint
+             frames stay aligned with the base frame. -->
+        <xacro:if value="${reflect}">
+            <xacro:property name="y_sign" value="-1"/>
+            <xacro:property name="mesh_roll" value="${pi}"/>
         </xacro:if>
-        <xacro:unless value="${(prefix == RL_) or (prefix == RR_)}">
-            <xacro:property name="hip_angle" value="0"/>
+        <xacro:unless value="${reflect}">
+            <xacro:property name="y_sign" value="1"/>
+            <xacro:property name="mesh_roll" value="0"/>
+        </xacro:unless>
+        <xacro:if value="${front}">
+            <xacro:property name="mesh_pitch" value="0"/>
+        </xacro:if>
+        <xacro:unless value="${front}">
+            <xacro:property name="mesh_pitch" value="${pi}"/>
         </xacro:unless>
         <joint name="${prefix}hip_joint" type="continuous">
@@ -29,5 +40,5 @@
             </inertial>
             <visual>
-                <origin xyz="0 0 0" rpy="0 0 0" />
+                <origin xyz="0 0 0" rpy="${mesh_roll} ${mesh_pitch} 0" />
                 <geometry>
                     <mesh filename="package://go2_description/meshes/leg/hip.dae" scale="1 1 1"/>
@@ -39,5 +50,5 @@
             </visual>
             <collision>
-                <origin xyz="0 0 0" rpy="0 0 0" />
+                <origin xyz="0 0 0" rpy="${mesh_roll} ${mesh_pitch} 0" />
                 <geometry>
                     <mesh filename="package://go2_description/meshes/leg/hip.dae" scale="1 1 1"/>
@@ -46,10 +57,5 @@
         </link>
         <xacro:go2_thigh prefix="${prefix}" parent="${prefix}hip_link" reflect="${reflect}">
-            <xacro:if value="${reflect}">
-                <origin xyz="${thigh_offset_x} ${thigh_offset_y} ${thigh_offset_z}" rpy="${PI} ${hip_angle} 0"/>
-            </xacro:if>
-            <xacro:unless value="${reflect}">
-                <origin xyz="${thigh_offset_x} ${thigh_offset_y} ${thigh_offset_z}" rpy="0 ${hip_angle} 0"/>
-            </xacro:unless>
+            <origin xyz="${thigh_offset_x} ${thigh_offset_y * y_sign} ${thigh_offset_z}" rpy="0 0 0"/>
         </xacro:go2_thigh>
     </xacro:macro>
