Commit message: fix: Add imu to prefixed joint and sensor names

File: urdf/sensors/imu.urdf.xacro (robot description, xacro)
@@ -2,5 +2,5 @@
 <robot name="imu_sensor" xmlns:xacro="http://wiki.ros.org/xacro">
   <xacro:macro name="imu_sensor" params="prefix parent *origin">
-	  <joint name="${prefix}_joint" type="fixed">
+	  <joint name="${prefix}imu_joint" type="fixed">
 	      <axis xyz="1 0 0"/>
 	      <xacro:insert_block name="origin"/>
@@ -25,8 +25,8 @@
 	  </link>
     <gazebo reference="${prefix}imu_link">
-      <sensor name="${prefix}_sensor" type="imu">
+      <sensor name="${prefix}imu_sensor" type="imu">
         <always_on>1</always_on>
         <update_rate>30</update_rate>
-        <topic>${prefix}/imu/data</topic>
+        <topic>${prefix}imu/data</topic>
       </sensor>
     </gazebo>
