Commit message: fix: Restore leg inertials and joint limits

File: urdf/leg/calf.urdf.xacro (robot description, xacro)
@@ -7,5 +7,11 @@
         <xacro:property name="foot_offset_y" value="0.0"/>
         <xacro:property name="foot_offset_z" value="-0.213"/>
-        <joint name="${prefix}calf_joint" type="continuous">
+        <xacro:if value="${reflect}">
+            <xacro:property name="y_sign" value="-1"/>
+        </xacro:if>
+        <xacro:unless value="${reflect}">
+            <xacro:property name="y_sign" value="1"/>
+        </xacro:unless>
+        <joint name="${prefix}calf_joint" type="revolute">
             <parent link="${parent}"/>
             <child link="${prefix}calf_link"/>
@@ -16,9 +22,9 @@
         <link name="${prefix}calf_link">
             <inertial>
-                <origin xyz="0 0 0" rpy="0 0 0" />
+                <origin xyz="0.00548 ${-0.000975 * y_sign} -0.115" rpy="0 0 0" />
                 <mass value="0.154" />
                 <inertia
-                    ixx="0.00108"   ixy="3.4E-07"   ixz="1.72E-05"
-                    iyy="0.0011"    iyz="8.28E-06"  izz="3.29E-05" />
+                    ixx="0.00108"   ixy="${3.4E-07 * y_sign}"   ixz="1.72E-05"
+                    iyy="0.0011"    iyz="${8.28E-06 * y_sign}"  izz="3.29E-05" />
             </inertial>
             <visual>

File: urdf/leg/hip.urdf.xacro (robot description, xacro)
@@ -7,7 +7,7 @@
         <xacro:property name="thigh_offset_y" value="0.0955"/>
         <xacro:property name="thigh_offset_z" value="0.0"/>
-        <!-- Mirror factors: y_sign flips left/right. The shared hip mesh is
-             reoriented per leg via the visual/collision origin only, so joint
-             frames stay aligned with the base frame. -->
+        <!-- Mirror factors: y_sign flips left/right, x_sign flips front/rear.
+             The shared hip mesh is reoriented per leg via the visual/collision
+             origin only, so joint frames stay aligned with the base frame. -->
         <xacro:if value="${reflect}">
             <xacro:property name="y_sign" value="-1"/>
@@ -19,10 +19,12 @@
         </xacro:unless>
         <xacro:if value="${front}">
+            <xacro:property name="x_sign" value="1"/>
             <xacro:property name="mesh_pitch" value="0"/>
         </xacro:if>
         <xacro:unless value="${front}">
+            <xacro:property name="x_sign" value="-1"/>
             <xacro:property name="mesh_pitch" value="${pi}"/>
         </xacro:unless>
-        <joint name="${prefix}hip_joint" type="continuous">
+        <joint name="${prefix}hip_joint" type="revolute">
             <parent link="${parent}"/>
             <child link="${prefix}hip_link"/>
@@ -33,9 +35,9 @@
         <link name="${prefix}hip_link">
             <inertial>
-                <origin xyz="0 0 0" rpy="0 0 0" />
-                <mass value="6.921" />
+                <origin xyz="${-0.0054 * x_sign} ${0.00194 * y_sign} -0.000105" rpy="0 0 0" />
+                <mass value="0.678" />
                 <inertia
-                    ixx="0.02448" ixy="0.00012166" ixz="0.0014849"
-                    iyy="0.098077" iyz="-3.12E-05" izz="0.107" />
+                    ixx="0.00048" ixy="${-3.01E-06 * x_sign * y_sign}" ixz="${1.11E-06 * x_sign}"
+                    iyy="0.000884" iyz="${-1.42E-06 * y_sign}" izz="0.000596" />
             </inertial>
             <visual>
@@ -56,5 +58,5 @@
             </collision>
         </link>
-        <xacro:go2_thigh prefix="${prefix}" parent="${prefix}hip_link" reflect="${reflect}">
+        <xacro:go2_thigh prefix="${prefix}" parent="${prefix}hip_link" front="${front}" reflect="${reflect}">
             <origin xyz="${thigh_offset_x} ${thigh_offset_y * y_sign} ${thigh_offset_z}" rpy="0 0 0"/>
         </xacro:go2_thigh>

File: urdf/leg/thigh.urdf.xacro (robot description, xacro)
@@ -3,22 +3,37 @@
 <xacro:include filename="$(find go2_description)/urdf/leg/calf.urdf.xacro"/>
     <!-- Define a macro for thigh -->
-    <xacro:macro name="go2_thigh" params="prefix parent *origin reflect">
+    <xacro:macro name="go2_thigh" params="prefix parent *origin front reflect">
         <xacro:property name="calf_offset_x" value="0.0"/>
         <xacro:property name="calf_offset_y" value="0.0"/>
         <xacro:property name="calf_offset_z" value="-0.213"/>
-        <joint name="${prefix}thigh_joint" type="continuous">
+        <xacro:if value="${reflect}">
+            <xacro:property name="y_sign" value="-1"/>
+        </xacro:if>
+        <xacro:unless value="${reflect}">
+            <xacro:property name="y_sign" value="1"/>
+        </xacro:unless>
+        <!-- Rear thighs have a wider extension range than front ones -->
+        <xacro:if value="${front}">
+            <xacro:property name="thigh_lower" value="-1.5708"/>
+            <xacro:property name="thigh_upper" value="3.4907"/>
+        </xacro:if>
+        <xacro:unless value="${front}">
+            <xacro:property name="thigh_lower" value="-0.5236"/>
+            <xacro:property name="thigh_upper" value="4.5379"/>
+        </xacro:unless>
+        <joint name="${prefix}thigh_joint" type="revolute">
             <parent link="${parent}"/>
             <child link="${prefix}thigh_link"/>
             <xacro:insert_block name="origin" />
             <axis xyz="0 1 0" />
-            <limit lower="-0.5236" upper="4.5379" effort="23.7" velocity="30.1" />
+            <limit lower="${thigh_lower}" upper="${thigh_upper}" effort="23.7" velocity="30.1" />
         </joint>
         <link name="${prefix}thigh_link">
             <inertial>
-                <origin xyz="0 0 0" rpy="0 0 0" />
+                <origin xyz="-0.00374 ${-0.0223 * y_sign} -0.0327" rpy="0 0 0" />
                 <mass value="1.152" />
                 <inertia
-                    ixx="0.00584"   ixy="8.72E-05"  ixz="-0.000289"
-                    iyy="0.0058"    iyz="0.000808"  izz="0.00103"  />
+                    ixx="0.00584"   ixy="${8.72E-05 * y_sign}"  ixz="-0.000289"
+                    iyy="0.0058"    iyz="${0.000808 * y_sign}"  izz="0.00103"  />
             </inertial>
             <visual>
