Commit message: refactor: Extract go2 body macro

File: robots/go2_description.urdf.xacro (robot description, xacro)
@@ -1,13 +1,8 @@
 <?xml version="1.0"?>
 <robot name="go2" xmlns:xacro="http://wiki.ros.org/xacro">
-<!-- Import elements (base + legs) -->
-<xacro:include filename="$(find go2_description)/urdf/base/base.urdf.xacro"/>
-<xacro:include filename="$(find go2_description)/urdf/base/leg.urdf.xacro"/>
+<!-- Import the Go2 body (base + legs) -->
+<xacro:include filename="$(find go2_description)/urdf/go2.urdf.xacro"/>
 <!-- Global Properties  -->
 <xacro:property name="PI" value="3.1415926535897931"/>
-<!-- Leg Allocations -->
-<xacro:property name="leg_offset_x" value="0.194"/>
-<xacro:property name="leg_offset_y" value="0.0465"/>
-<xacro:property name="leg_offset_z" value="0.0"/>
 <!-- Arguments -->
 <xacro:arg name="prefix" default=""/>
@@ -37,18 +32,5 @@
   <origin xyz="0.15 0 0.12" rpy="0 0 ${PI/2}"/>
 </xacro:hesai_sensor>
-<!-- Robot base -->
-<xacro:go2_base prefix="$(arg prefix)"/>
-<!-- Legs -->
-<xacro:go2_leg prefix="FL_" parent="$(arg prefix)base_link" reflect="false"
-        x="${leg_offset_x}"   y="${leg_offset_y}"   z="${leg_offset_z}"
-        roll="0"      pitch="0"   yaw="0"/>
-<xacro:go2_leg prefix="FR_" parent="$(arg prefix)base_link" reflect="true"
-        x="${leg_offset_x}"   y="-${leg_offset_y}"  z="${leg_offset_z}"
-        roll="${PI}"  pitch="0"   yaw="0"/>
-<xacro:go2_leg prefix="RL_" parent="$(arg prefix)base_link" reflect="false"
-        x="-${leg_offset_x}"  y="${leg_offset_y}"   z="${leg_offset_z}"
-        roll="${PI}"  pitch="0"   yaw="${PI}"/>
-<xacro:go2_leg prefix="RR_" parent="$(arg prefix)base_link" reflect="true"
-        x="-${leg_offset_x}"  y="-${leg_offset_y}"  z="${leg_offset_z}"
-        roll="0"      pitch="0"   yaw="${PI}"/>
+<!-- Robot body (base + legs) -->
+<xacro:go2 prefix="$(arg prefix)"/>
 </robot>

Commit message: refactor: Move built-in sensors into go2 macro

File: robots/go2_description.urdf.xacro (robot description, xacro)
@@ -12,19 +12,6 @@
 <xacro:arg name="name" default="go2"/>
 <!-- Sensors -->
-<!-- IMU -->
-<xacro:include filename="$(find go2_description)/urdf/sensors/imu.urdf.xacro"/>
-<xacro:imu_sensor prefix="$(arg prefix)" parent="$(arg prefix)base_link">
-  <origin xyz="-0.02557 0 0.04232" rpy="0 0 0"/>
-</xacro:imu_sensor>
-<!-- camera -->
-<xacro:include filename="$(find go2_description)/urdf/sensors/camera.urdf.xacro"/>
-<xacro:camera_sensor prefix="$(arg prefix)" parent="$(arg prefix)base_link">
-  <origin xyz="0.325 0 0.045" rpy="0 0 0"/>
-</xacro:camera_sensor>
-<!-- radar -->
-<xacro:include filename="$(find go2_description)/urdf/sensors/radar.urdf.xacro"/>
-<xacro:radar_sensor prefix="$(arg prefix)" parent="$(arg prefix)base_link">
-  <origin xyz="0.28945 0 -0.046825" rpy="0 2.8782 0"/>
-</xacro:radar_sensor>
+<!-- Built-in sensors (IMU, front camera, L1 lidar) are defined inside the
+     go2 macro. Only optional external sensors are added here. -->
 <!-- hesai lidar -->
 <xacro:include filename="$(find go2_description)/urdf/sensors/hesai.urdf.xacro"/>

File: urdf/go2.urdf.xacro (robot description, xacro)
@@ -1,7 +1,11 @@
 <?xml version="1.0"?>
 <robot name="go2" xmlns:xacro="http://www.ros.org/wiki/xacro">
-<!-- Import elements (base + legs) -->
+<!-- Import elements (base + legs + built-in sensors) -->
 <xacro:include filename="$(find go2_description)/urdf/base/base.urdf.xacro"/>
 <xacro:include filename="$(find go2_description)/urdf/base/leg.urdf.xacro"/>
+<xacro:include filename="$(find go2_description)/urdf/sensors/imu.urdf.xacro"/>
+<xacro:include filename="$(find go2_description)/urdf/sensors/camera.urdf.xacro"/>
+<!-- Required by the camera macro -->
+<xacro:property name="PI" value="${pi}"/>
 <!-- Define a macro for the whole Go2 body (base + legs) -->
 <xacro:macro name="go2" params="prefix">
@@ -22,4 +26,28 @@
     <xacro:go2_leg prefix="${prefix}RR_" parent="${prefix}base_link" front="false" reflect="true"
             x="-${leg_offset_x}"  y="-${leg_offset_y}"  z="${leg_offset_z}"/>
+    <!-- Built-in IMU. The go2_ prefix avoids clashing with external IMUs. -->
+    <xacro:imu_sensor prefix="${prefix}go2_" parent="${prefix}base_link">
+        <origin xyz="-0.02557 0 0.04232" rpy="0 0 0"/>
+    </xacro:imu_sensor>
+    <!-- Built-in front camera. The go2_ prefix avoids clashing with external
+         cameras. -->
+    <xacro:camera_sensor prefix="${prefix}go2_" parent="${prefix}base_link">
+        <origin xyz="0.325 0 0.045" rpy="0 0 0"/>
+    </xacro:camera_sensor>
+    <!-- Unitree 4D LiDAR-L1. Frame names are fixed by the Go2 firmware,
+         so no prefix is applied. -->
+    <link name="utlidar_lidar"/>
+    <joint name="base_to_utlidar_lidar" type="fixed">
+        <parent link="${prefix}base_link"/>
+        <child link="utlidar_lidar"/>
+        <origin xyz="0.28945 0 -0.046825" rpy="0 2.8782 0"/>
+    </joint>
+    <!-- The L1 IMU axes are parallel to the L1 point cloud frame. -->
+    <link name="utlidar_imu"/>
+    <joint name="utlidar_lidar_to_utlidar_imu" type="fixed">
+        <parent link="utlidar_lidar"/>
+        <child link="utlidar_imu"/>
+        <origin xyz="0 0 0" rpy="0 0 0"/>
+    </joint>
 </xacro:macro>
 </robot>

Commit message: refactor: Use xacro built-in pi instead of PI property

File: robots/go2_description.urdf.xacro (robot description, xacro)
@@ -3,6 +3,4 @@
 <!-- Import the Go2 body (base + legs) -->
 <xacro:include filename="$(find go2_description)/urdf/go2.urdf.xacro"/>
-<!-- Global Properties  -->
-<xacro:property name="PI" value="3.1415926535897931"/>
 <!-- Arguments -->
 <xacro:arg name="prefix" default=""/>
@@ -13,5 +11,5 @@
 <xacro:include filename="$(find go2_description)/urdf/sensors/hesai.urdf.xacro"/>
 <xacro:hesai_sensor prefix="$(arg prefix)" parent="$(arg prefix)base_link">
-  <origin xyz="0.15 0 0.12" rpy="0 0 ${PI/2}"/>
+  <origin xyz="0.15 0 0.12" rpy="0 0 ${pi/2}"/>
 </xacro:hesai_sensor>
 <!-- Robot body (base + legs) -->

File: urdf/go2.urdf.xacro (robot description, xacro)
@@ -6,6 +6,4 @@
 <xacro:include filename="$(find go2_description)/urdf/sensors/imu.urdf.xacro"/>
 <xacro:include filename="$(find go2_description)/urdf/sensors/camera.urdf.xacro"/>
-<!-- Required by the camera macro -->
-<xacro:property name="PI" value="${pi}"/>
 <!-- Define a macro for the whole Go2 body (base + legs) -->
 <xacro:macro name="go2" params="prefix">

File: urdf/sensors/camera.urdf.xacro (robot description, xacro)
@@ -27,5 +27,5 @@
             <parent link="${prefix}camera_link"/>
             <child link="${prefix}camera_optical_frame"/>
-            <origin xyz="0 0 0" rpy="-${PI/2} 0 -${PI/2}" />
+            <origin xyz="0 0 0" rpy="-${pi/2} 0 -${pi/2}" />
         </joint>
         <link name="${prefix}camera_optical_frame">

Commit message: refactor: Drop dead prefix plumbing from the go2 macro

File: robots/go2_description.urdf.xacro (robot description, xacro)
@@ -12,4 +12,4 @@
 </xacro:hesai_sensor>
 <!-- Robot body (base + legs) -->
-<xacro:go2 prefix=""/>
+<xacro:go2/>
 </robot>

File: urdf/go2.urdf.xacro (robot description, xacro)
@@ -7,5 +7,5 @@
 <xacro:include filename="$(find go2_description)/urdf/sensors/camera.urdf.xacro"/>
 <!-- Define a macro for the whole Go2 body (base + legs) -->
-<xacro:macro name="go2" params="prefix">
+<xacro:macro name="go2">
     <!-- Leg Allocations -->
     <xacro:property name="leg_offset_x" value="0.1934"/>
@@ -13,29 +13,28 @@
     <xacro:property name="leg_offset_z" value="0.0"/>
     <!-- Robot base -->
-    <xacro:go2_base prefix="${prefix}"/>
+    <xacro:go2_base prefix=""/>
     <!-- Legs: front/left flags select joint limits, inertia mirroring and meshes.
          All joint origins are pure translations (no rotation), matching the real robot. -->
-    <xacro:go2_leg prefix="${prefix}FL_" parent="${prefix}base_link" front="true" reflect="false"
+    <xacro:go2_leg prefix="FL_" parent="base_link" front="true" reflect="false"
             x="${leg_offset_x}"   y="${leg_offset_y}"   z="${leg_offset_z}"/>
-    <xacro:go2_leg prefix="${prefix}FR_" parent="${prefix}base_link" front="true" reflect="true"
+    <xacro:go2_leg prefix="FR_" parent="base_link" front="true" reflect="true"
             x="${leg_offset_x}"   y="-${leg_offset_y}"  z="${leg_offset_z}"/>
-    <xacro:go2_leg prefix="${prefix}RL_" parent="${prefix}base_link" front="false" reflect="false"
+    <xacro:go2_leg prefix="RL_" parent="base_link" front="false" reflect="false"
             x="-${leg_offset_x}"  y="${leg_offset_y}"   z="${leg_offset_z}"/>
-    <xacro:go2_leg prefix="${prefix}RR_" parent="${prefix}base_link" front="false" reflect="true"
+    <xacro:go2_leg prefix="RR_" parent="base_link" front="false" reflect="true"
             x="-${leg_offset_x}"  y="-${leg_offset_y}"  z="${leg_offset_z}"/>
     <!-- Built-in IMU. The go2_ prefix avoids clashing with external IMUs. -->
-    <xacro:imu_sensor prefix="${prefix}go2_" parent="${prefix}base_link">
+    <xacro:imu_sensor prefix="go2_" parent="base_link">
         <origin xyz="-0.02557 0 0.04232" rpy="0 0 0"/>
     </xacro:imu_sensor>
     <!-- Built-in front camera. The go2_ prefix avoids clashing with external
          cameras. -->
-    <xacro:camera_sensor prefix="${prefix}go2_" parent="${prefix}base_link">
+    <xacro:camera_sensor prefix="go2_" parent="base_link">
         <origin xyz="0.325 0 0.045" rpy="0 0 0"/>
     </xacro:camera_sensor>
-    <!-- Unitree 4D LiDAR-L1. Frame names are fixed by the Go2 firmware,
-         so no prefix is applied. -->
+    <!-- Unitree 4D LiDAR-L1. Frame names are fixed by the Go2 firmware. -->
     <link name="utlidar_lidar"/>
     <joint name="base_to_utlidar_lidar" type="fixed">
-        <parent link="${prefix}base_link"/>
+        <parent link="base_link"/>
         <child link="utlidar_lidar"/>
         <origin xyz="0.28945 0 -0.046825" rpy="0 2.8782 0"/>

Commit message: refactor: Drop meaningless prefix params from base and hesai macros

File: robots/go2_description.urdf.xacro (robot description, xacro)
@@ -8,5 +8,5 @@
 <!-- hesai lidar -->
 <xacro:include filename="$(find go2_description)/urdf/sensors/hesai.urdf.xacro"/>
-<xacro:hesai_sensor prefix="" parent="base_link">
+<xacro:hesai_sensor parent="base_link">
   <origin xyz="0.15 0 0.12" rpy="0 0 ${pi/2}"/>
 </xacro:hesai_sensor>

File: urdf/base/base.urdf.xacro (robot description, xacro)
@@ -2,6 +2,6 @@
 <robot name="base" xmlns:xacro="http://www.ros.org/wiki/xacro">
     <!-- Define a macro for base_link -->
-    <xacro:macro name="go2_base" params="prefix">
-        <link name="${prefix}base_link">
+    <xacro:macro name="go2_base">
+        <link name="base_link">
             <inertial>
                 <origin xyz="0.021112 0 -0.005366" rpy="0 0 0" />

File: urdf/go2.urdf.xacro (robot description, xacro)
@@ -13,5 +13,5 @@
     <xacro:property name="leg_offset_z" value="0.0"/>
     <!-- Robot base -->
-    <xacro:go2_base prefix=""/>
+    <xacro:go2_base/>
     <!-- Legs: front/left flags select joint limits, inertia mirroring and meshes.
          All joint origins are pure translations (no rotation), matching the real robot. -->

File: urdf/sensors/hesai.urdf.xacro (robot description, xacro)
@@ -2,11 +2,11 @@
 <robot xmlns:xacro="http://www.ros.org/wiki/xacro" name="hesai_sensor">
     <!-- Hesai Sensor Macro -->
-    <xacro:macro name="hesai_sensor" params="prefix parent *origin">
-        <joint name="${prefix}lidar_joint" type="fixed">
+    <xacro:macro name="hesai_sensor" params="parent *origin">
+        <joint name="lidar_joint" type="fixed">
             <parent link="${parent}"/>
-            <child link="${prefix}lidar_link"/>
+            <child link="lidar_link"/>
             <xacro:insert_block name="origin" />
         </joint>
-        <link name="${prefix}lidar_link">
+        <link name="lidar_link">
             <visual>
                 <geometry>
@@ -28,10 +28,10 @@
             </inertial>
         </link>
-        <gazebo reference="${prefix}lidar_link">
+        <gazebo reference="lidar_link">
             <sensor name='gpu_lidar' type='gpu_lidar'>
-            <pose relative_to="${prefix}lidar_link">0 0 0 0 0 0</pose>
-            <topic>${prefix}lidar_sensor</topic>
+            <pose relative_to="lidar_link">0 0 0 0 0 0</pose>
+            <topic>lidar_sensor</topic>
             <update_rate>20</update_rate>
-            <gz_frame_id>${prefix}lidar_link</gz_frame_id>
+            <gz_frame_id>lidar_link</gz_frame_id>
             <lidar>
                 <scan>
